File: PCB/agricoltura-SunLeaf-2.4G/agricoltura-SunLeaf-2.4G.kicad_pcb (KiCad board)
At the start: 4 copper layers, 100 x 40 mm, 90 parts, among them M1 STM32WB5MMGH6TR, Q1 DMP3125L-7, Q2 DMP3125L-7, SW1 B3U-1000P, T1 B2B-PH-K-S(LF)(SN), T10 BM04B-SRSS-TB(LF)(SN), T11 BM04B-SRSS-TB(LF)(SN), T12 BM04B-SRSS-TB(LF)(SN), T13 BM04B-SRSS-TB(LF)(SN), T14 BM04B-SRSS-TB(LF)(SN)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

Commit message: KiCAD 8
Projected updated to KiCAD 8
Other:
- net class Default removed
